Commit message: Tweezer and scalpel setup in there with a rotation stage for the sample holder

File: urdf/materials.xacro (robot description, xacro)
@@ -1,4 +1,4 @@
 <?xml version="1.0" ?>
-<robot name="linear_stage" xmlns:xacro="http://www.ros.org/wiki/xacro" >
+<robot name="stage" xmlns:xacro="http://www.ros.org/wiki/xacro" >
 <material name="silver">
   <color rgba="0.700 0.700 0.700 1.000"/>

File: urdf/single_stage.urdf.xacro (robot description, xacro)
@@ -2,15 +2,22 @@
 <robot xmlns:xacro="http://www.ros.org/wiki/xacro" name="iiwa">
     <xacro:arg name="hardware_interface" default="PositionJointInterface"/>
-    <xacro:arg name="initial_z" default="0.0"/>
+    <xacro:property name="type" value="rot"/>
+    <xacro:arg name="prefix" default="x"/>
     <link name="base_link"/>
-    <xacro:include filename="$(find micro_resector_description)/urdf/linear_stage.xacro"/>
-    <xacro:arg name="prefix" default="x"/>
-    <xacro:arg name="hardware_interface" default="PositionJointInterface"/>
-    <joint name="$(arg prefix)_linear_stage_world_joint" type="fixed">
+    <xacro:include filename="$(find micro_resector_description)/urdf/materials.xacro" />
+    <xacro:include filename="$(find micro_resector_description)/urdf/stage/linear_stage.xacro"/>
+    <xacro:include filename="$(find micro_resector_description)/urdf/stage/rotation_stage.xacro"/>
+    <joint name="$(arg prefix)_${type}_stage_world_joint" type="fixed">
         <parent link="base_link"/>
-        <child link="$(arg prefix)_base_link"/>
+        <child link="$(arg prefix)_${type}_base_link"/>
         <origin xyz="0.0 0.0 0.00" rpy="${pi/2} 0.0 0.0"/>
     </joint>
-    <xacro:linear_stage hardware_interface="$(arg hardware_interface)" prefix="$(arg prefix)">
-    </xacro:linear_stage>
+    <xacro:if value="${type == 'lin'}">
+        <xacro:linear_stage hardware_interface="$(arg hardware_interface)" prefix="$(arg prefix)">
+        </xacro:linear_stage>
+    </xacro:if>
+    <xacro:if value="${type == 'rot'}">
+        <xacro:rotation_stage hardware_interface="$(arg hardware_interface)" prefix="$(arg prefix)">
+        </xacro:rotation_stage>
+    </xacro:if>
 </robot>

File: urdf/stage/linear_stage.xacro (robot description, xacro)
@@ -1,9 +1,8 @@
 <?xml version="1.0" ?>
 <robot name="linear_stage" xmlns:xacro="http://www.ros.org/wiki/xacro">
-<xacro:include filename="$(find micro_resector_description)/urdf/materials.xacro" />
-<xacro:include filename="$(find micro_resector_description)/urdf/linear_stage.trans" />
-<xacro:include filename="$(find micro_resector_description)/urdf/linear_stage.gazebo" />
+<xacro:include filename="$(find micro_resector_description)/urdf/stage/stage.trans" />
+<xacro:include filename="$(find micro_resector_description)/urdf/stage/stage.gazebo" />
 <xacro:macro name="linear_stage" params="prefix hardware_interface">
-  <link name="${prefix}_base_link">
+  <link name="${prefix}_lin_base_link">
     <inertial>
       <origin rpy="0 0 0" xyz="0.0 0.0015 0.0"/>
@@ -14,5 +13,5 @@
       <origin rpy="0 0 0" xyz="0 0.0095 0"/>
       <geometry>
-        <mesh filename="package://micro_resector_description/meshes/lin_base_link.stl" scale="0.001 0.001 0.001"/>
+        <mesh filename="package://micro_resector_description/meshes/stage/lin_base_link.stl" scale="0.001 0.001 0.001"/>
       </geometry>
       <material name="silver"/>
@@ -21,9 +20,9 @@
       <origin rpy="0 0 0" xyz="0 0.0095 0"/>
       <geometry>
-        <mesh filename="package://micro_resector_description/meshes/lin_base_link.stl" scale="0.001 0.001 0.001"/>
+        <mesh filename="package://micro_resector_description/meshes/stage/lin_base_link.stl" scale="0.001 0.001 0.001"/>
       </geometry>
     </collision>
   </link>
-  <link name="${prefix}_stage_link">
+  <link name="${prefix}_lin_stage_link">
     <inertial>
       <origin rpy="0 0 0" xyz="0.0 -0.00028 0.0"/>
@@ -34,5 +33,5 @@
       <origin rpy="0 0 0" xyz="0.0 0.0 -0.0"/>
       <geometry>
-        <mesh filename="package://micro_resector_description/meshes/lin_stage_link.stl" scale="0.001 0.001 0.001"/>
+        <mesh filename="package://micro_resector_description/meshes/stage/lin_stage_link.stl" scale="0.001 0.001 0.001"/>
       </geometry>
       <material name="silver"/>
@@ -41,17 +40,17 @@
       <origin rpy="0 0 0" xyz="0.0 0.0 -0.0"/>
       <geometry>
-        <mesh filename="package://micro_resector_description/meshes/lin_stage_link.stl" scale="0.001 0.001 0.001"/>
+        <mesh filename="package://micro_resector_description/meshes/stage/lin_stage_link.stl" scale="0.001 0.001 0.001"/>
       </geometry>
     </collision>
   </link>
-  <joint name="${prefix}_joint" type="prismatic">
+  <joint name="${prefix}_lin_joint" type="prismatic">
     <origin rpy="0 0 0" xyz="0.0 0.0095 0.0"/>
-    <parent link="${prefix}_base_link"/>
-    <child link="${prefix}_stage_link"/>
+    <parent link="${prefix}_lin_base_link"/>
+    <child link="${prefix}_lin_stage_link"/>
     <axis xyz="1 0.0 0.0"/>
     <limit effort="100" lower="-0.015" upper="0.015" velocity="0.0045"/>
   </joint>
-  <xacro:linear_stage_gazebo prefix="$(arg prefix)"/>
-  <xacro:linear_stage_transmission prefix="$(arg prefix)" hardware_interface="${hardware_interface}"/>
+  <xacro:stage_gazebo prefix="$(arg prefix)" type="lin"/>
+  <xacro:stage_transmission prefix="$(arg prefix)" hardware_interface="${hardware_interface}" type="lin"/>
 </xacro:macro>
 </robot>

File: urdf/xyz_stage.urdf.xacro (robot description, xacro)
@@ -6,4 +6,5 @@
     <xacro:include filename="$(find micro_resector_description)/urdf/materials.xacro" />
     <xacro:include filename="$(find micro_resector_description)/urdf/stage/linear_stage.xacro"/>
+    <xacro:include filename="$(find micro_resector_description)/urdf/link/l_bracket.xacro"/>
     <joint name="x_linear_stage_world_joint" type="fixed">
         <parent link="base_link"/>
@@ -13,5 +14,5 @@
     <xacro:linear_stage hardware_interface="$(arg hardware_interface)" prefix="x">
     </xacro:linear_stage>
-    <joint name="y_linear_stage_world_joint" type="fixed">
+    <joint name="y_linear_stage_joint" type="fixed">
         <parent link="x_lin_stage_link"/>
         <child link="y_lin_base_link"/>
@@ -20,3 +21,17 @@
     <xacro:linear_stage hardware_interface="$(arg hardware_interface)" prefix="y">
     </xacro:linear_stage>
+    <joint name="l_bracket_joint" type="fixed">
+        <parent link="y_lin_stage_link"/>
+        <child link="z_bracket_base_link"/>
+        <origin xyz="0.0 0.0 0.00" rpy="0.0 0.0 0.0"/>
+    </joint>
+    <xacro:l_bracket prefix="z">
+    </xacro:l_bracket>
+    <joint name="z_linear_stage_joint" type="fixed">
+        <parent link="z_bracket_side_link"/>
+        <child link="z_lin_base_link"/>
+        <origin xyz="0.0 0.0 0.00" rpy="0.0 ${pi/2} 0.0"/>
+    </joint>
+    <xacro:linear_stage hardware_interface="$(arg hardware_interface)" prefix="z">
+    </xacro:linear_stage>
 </robot>
