Commit message: added properties for each device to make setup easier

File: urdf/micro_resector.ros2_control.xacro (robot description, xacro)
@@ -3,4 +3,7 @@
     <xacro:macro name="micro_resector_control" params="name hardware:=false">
         <xacro:property name="linear_position_limit" value="0.015"/>
+        <xacro:property name="tweezer_device" value="2"/>
+        <xacro:property name="scalpel_device" value="3"/>
+        <xacro:property name="sample_holder_device" value="1"/>
         <ros2_control name="${name}" type="system">
             <hardware>
@@ -20,5 +23,5 @@
                 <state_interface name="velocity"/>
                 <xacro:if value="${hardware}">
-                    <param name="device">2</param>
+                    <param name="device">${tweezer_device}</param>
                     <param name="axis">0</param>
                     <param name="type">6</param>
@@ -35,5 +38,5 @@
                 <state_interface name="velocity"/>
                 <xacro:if value="${hardware}">
-                    <param name="device">2</param>
+                    <param name="device">${tweezer_device}</param>
                     <param name="axis">1</param>
                     <param name="type">6</param>
@@ -50,5 +53,5 @@
                 <state_interface name="velocity"/>
                 <xacro:if value="${hardware}">
-                    <param name="device">2</param>
+                    <param name="device">${tweezer_device}</param>
                     <param name="axis">2</param>
                     <param name="type">6</param>
@@ -65,5 +68,5 @@
                 <state_interface name="velocity"/>
                 <xacro:if value="${hardware}">
-                    <param name="device">0</param>
+                    <param name="device">${scalpel_device}</param>
                     <param name="axis">0</param>
                     <param name="type">6</param>
@@ -80,5 +83,5 @@
                 <state_interface name="velocity"/>
                 <xacro:if value="${hardware}">
-                    <param name="device">0</param>
+                    <param name="device">${scalpel_device}</param>
                     <param name="axis">1</param>
                     <param name="type">6</param>
@@ -95,5 +98,5 @@
                 <state_interface name="velocity"/>
                 <xacro:if value="${hardware}">
-                    <param name="device">0</param>
+                    <param name="device">${scalpel_device}</param>
                     <param name="axis">2</param>
                     <param name="type">6</param>
@@ -107,5 +110,5 @@
                 <state_interface name="velocity"/>
                 <xacro:if value="${hardware}">
-                    <param name="device">1</param>
+                    <param name="device">${sample_holder_device}</param>
                     <param name="axis">0</param>
                     <param name="type">14</param>
