Commit message: moved to new tweezer and scalpel designs and link naming conventions for the tools

File: urdf/scalpel_system.xacro (robot description, xacro)
@@ -4,4 +4,5 @@
     <xacro:include filename="$(find micro_resector_description)/urdf/link/l_bracket.xacro"/>
     <xacro:include filename="$(find micro_resector_description)/urdf/tools/scalpel.xacro"/>
+    <xacro:include filename="$(find micro_resector_description)/urdf/tools/scalpel_assembly.xacro"/>
     <xacro:include filename="$(find micro_resector_description)/urdf/tools/tool_holder.xacro"/>
     <xacro:macro name="scalpel_system" params="hardware_interface name">
@@ -38,18 +39,25 @@
         <xacro:linear_stage hardware_interface="${hardware_interface}" prefix="${name}_z">
         </xacro:linear_stage>
-        <joint name="${name}_tool_holder_joint" type="fixed">-->
+        <xacro:scalpel_assembly>
+        </xacro:scalpel_assembly>
+        <joint name="scalpel_assembly_joint" type="fixed">
             <parent link="${name}_z_lin_stage_link"/>
-            <child link="${name}_tool_holder_link"/>
-            <origin xyz="0 0 0" rpy="0 0 ${pi/2}"/>
+            <child link="scalpel_tool_holder_link"/>
+            <origin xyz="0 0 0" rpy="${-pi/2} 0 ${pi/2}"/>
         </joint>
-        <xacro:tool_holder name="${name}">
-        </xacro:tool_holder>
-        <joint name="${name}_attachment_joint" type="fixed">
-            <parent link="${name}_tool_attachment_link"/>
-            <child link="scalpel_z_scalpel_base_link"/>
-            <origin xyz="0.0 0.0 0.00" rpy="0.0 0.0 0.0"/>
-        </joint>
-        <xacro:scalpel prefix="scalpel_z">
-        </xacro:scalpel>
+<!--        <joint name="${name}_tool_holder_joint" type="fixed">&ndash;&gt;-->
+<!--            <parent link="${name}_z_lin_stage_link"/>-->
+<!--            <child link="${name}_tool_holder_link"/>-->
+<!--            <origin xyz="0 0 0" rpy="0 0 ${pi/2}"/>-->
+<!--        </joint>-->
+<!--        <xacro:tool_holder name="${name}">-->
+<!--        </xacro:tool_holder>-->
+<!--        <joint name="${name}_attachment_joint" type="fixed">-->
+<!--            <parent link="${name}_tool_attachment_link"/>-->
+<!--            <child link="scalpel_z_scalpel_base_link"/>-->
+<!--            <origin xyz="0.0 0.0 0.00" rpy="0.0 0.0 0.0"/>-->
+<!--        </joint>-->
+<!--        <xacro:scalpel prefix="scalpel_z">-->
+<!--        </xacro:scalpel>-->
     </xacro:macro>
 </robot>

File: urdf/tweezer_system.xacro (robot description, xacro)
@@ -4,5 +4,5 @@
     <xacro:include filename="$(find micro_resector_description)/urdf/link/l_bracket.xacro"/>
     <xacro:include filename="$(find micro_resector_description)/urdf/tools/tweezer_reinforced.xacro"/>
-    <xacro:include filename="$(find micro_resector_description)/urdf/tools/tool_holder.xacro"/>
+    <xacro:include filename="$(find micro_resector_description)/urdf/tools/tweezer_assembly.xacro"/>
     <xacro:macro name="tweezer_system" params="hardware_interface name">
 <!--        <xacro:arg name="hardware_interface" default="PositionJointInterface"/>-->
@@ -38,18 +38,11 @@
         <xacro:linear_stage hardware_interface="${hardware_interface}" prefix="${name}_z">
         </xacro:linear_stage>
-        <joint name="${name}_tool_holder_joint" type="fixed">-->
+        <xacro:tweezer_assembly>
+        </xacro:tweezer_assembly>
+        <joint name="tweezer_assembly_joint" type="fixed">
             <parent link="${name}_z_lin_stage_link"/>
-            <child link="${name}_tool_holder_link"/>
-            <origin xyz="0 0 0.006" rpy="0 ${pi} ${pi/2}"/>
+            <child link="tweezer_tool_holder_link"/>
+            <origin xyz="0 0 0" rpy="${-pi/2} 0 ${pi/2}"/>
         </joint>
-        <xacro:tool_holder name="${name}">
-        </xacro:tool_holder>
-        <joint name="${name}_attachment_joint" type="fixed">
-            <parent link="${name}_tool_attachment_link"/>
-            <child link="tweezer_z_tweezer_base_link"/>
-            <origin xyz="0.0 0.0 0.00" rpy="0.0 0.0 0.0"/>
-        </joint>
-        <xacro:tweezer prefix="tweezer_z">
-        </xacro:tweezer>
     </xacro:macro>
 </robot>
