Commit message: Added colours to the main componets added a sample holder xacro with rot stage and box

File: urdf/full_setup.urdf.xacro (robot description, xacro)
@@ -7,5 +7,5 @@
     <xacro:include filename="$(find micro_resector_description)/urdf/tweezer_system.xacro" />
     <xacro:include filename="$(find micro_resector_description)/urdf/scalpel_system.xacro"/>
-    <xacro:include filename="$(find micro_resector_description)/urdf/stage/rotation_stage.xacro"/>
+    <xacro:include filename="$(find micro_resector_description)/urdf/sample_holder_system.xacro"/>
     <joint name="tweezer_to_base" type="fixed">
         <parent link="base_link"/>
@@ -22,10 +22,10 @@
     <xacro:scalpel_system hardware_interface="$(arg hardware_interface)">
     </xacro:scalpel_system>
-    <joint name="rotation_stage_to_base" type="fixed">
+    <joint name="sample_holder_to_base" type="fixed">
         <parent link="base_link"/>
-        <child link="centre_rot_base_link"/>
-        <origin xyz="0 0 0.00" rpy="${pi/2} 0.0 0.0"/>
+        <child link="sample_holder_base_link"/>
+        <origin xyz="0 0 0.00" rpy="0 0.0 0.0"/>
     </joint>
-    <xacro:rotation_stage hardware_interface="$(arg hardware_interface)" prefix="centre">
-    </xacro:rotation_stage>
+    <xacro:sample_holder hardware_interface="$(arg hardware_interface)">
+    </xacro:sample_holder>
 </robot>

File: urdf/materials.xacro (robot description, xacro)
@@ -1,6 +1,30 @@
 <?xml version="1.0" ?>
-<robot name="stage" xmlns:xacro="http://www.ros.org/wiki/xacro" >
-<material name="silver">
-  <color rgba="0.700 0.700 0.700 1.000"/>
-</material>
+<robot name="materials" xmlns:xacro="http://www.ros.org/wiki/xacro" >
+  <material name="silver">
+    <color rgba="0.700 0.700 0.700 1.000"/>
+  </material>
+  <material name="black">
+    <color rgba="0.0 0.0 0.0 1.0"/>
+  </material>
+  <material name="blue">
+    <color rgba="0.0 0.0 0.8 1.0"/>
+  </material>
+  <material name="green">
+    <color rgba="0.0 0.8 0.0 1.0"/>
+  </material>
+  <material name="grey">
+    <color rgba="0.4 0.4 0.4 1.0"/>
+  </material>
+  <material name="orange">
+    <color rgba="${255/255} ${108/255} ${10/255} 1.0"/>
+  </material>
+  <material name="brown">
+    <color rgba="${222/255} ${207/255} ${195/255} 1.0"/>
+  </material>
+  <material name="red">
+    <color rgba="0.8 0.0 0.0 1.0"/>
+  </material>
+  <material name="white">
+    <color rgba="1.0 1.0 1.0 1.0"/>
+  </material>
 </robot>

File: urdf/tools/scalpel.xacro (robot description, xacro)
@@ -13,5 +13,5 @@
         <mesh filename="package://micro_resector_description/meshes/tools/scalpel.stl" scale="0.001 0.001 0.001"/>
       </geometry>
-      <material name="silver"/>
+      <material name="blue"/>
     </visual>
     <collision>

File: urdf/tools/tweezer.xacro (robot description, xacro)
@@ -10,5 +10,5 @@
           <mesh filename="package://micro_resector_description/meshes/tools/tweezer_left.stl" scale="0.001 0.001 0.001"/>
         </geometry>
-        <material name="silver"/>
+        <material name="red"/>
       </visual>
       <collision>
@@ -33,5 +33,5 @@
           <mesh filename="package://micro_resector_description/meshes/tools/tweezer_right.stl" scale="0.001 0.001 0.001"/>
         </geometry>
-        <material name="silver"/>
+        <material name="green"/>
       </visual>
       <collision>

Commit message: Added camera to gazebo sim.

File: urdf/full_setup.urdf.xacro (robot description, xacro)
@@ -8,4 +8,5 @@
     <xacro:include filename="$(find micro_resector_description)/urdf/scalpel_system.xacro"/>
     <xacro:include filename="$(find micro_resector_description)/urdf/sample_holder_system.xacro"/>
+    <xacro:include filename="$(find micro_resector_description)/urdf/tools/microscope_camera.xacro"/>
     <joint name="tweezer_to_base" type="fixed">
         <parent link="base_link"/>
@@ -29,3 +30,10 @@
     <xacro:sample_holder hardware_interface="$(arg hardware_interface)">
     </xacro:sample_holder>
+    <joint name="camera_joint" type="fixed">
+        <origin xyz="0 0 0.1" rpy="0 ${pi/2} 0"/>
+        <parent link="base_link"/>
+        <child link="camera_link"/>
+    </joint>
+    <xacro:microscope_camera type="mono"/>
+    <xacro:include filename="$(find micro_resector_description)/urdf/full_setup.gazebo.xacro"/>
 </robot>

File: urdf/materials.xacro (robot description, xacro)
@@ -28,6 +28,3 @@
     <color rgba="1.0 1.0 1.0 1.0"/>
   </material>
-  <gazebo>
-    <plugin filename="libgazebo_ros_control.so" name="control"/>
-  </gazebo>
 </robot>

Commit message: Added brainslice mock up scaled to double size. Fits with current instruments but will need to look into the instrument scales.

File: urdf/full_setup.urdf.xacro (robot description, xacro)
@@ -36,4 +36,10 @@
     </joint>
     <xacro:microscope_camera type="mono"/>
+    <joint name="sample_joint" type="fixed">
+        <parent link="sample_link"/>
+        <child link="brain_slice_base_link"/>
+        <origin xyz="0 0.0 0.00" rpy="0 0.0 0.0"/>
+    </joint>
+    <xacro:include filename="$(find micro_resector_description)/urdf/samples/brain_slice.urdf.xacro"/>
     <xacro:include filename="$(find micro_resector_description)/urdf/full_setup.gazebo.xacro"/>
 </robot>

Commit message: Modified end links so z is up

File: urdf/full_setup.urdf.xacro (robot description, xacro)
@@ -39,5 +39,5 @@
         <parent link="sample_link"/>
         <child link="brain_slice_base_link"/>
-        <origin xyz="0 0.0 0.00" rpy="0 0.0 0.0"/>
+        <origin xyz="0 0.0 0.0005" rpy="0 0.0 0.0"/>
     </joint>
     <xacro:include filename="$(find micro_resector_description)/urdf/samples/brain_slice.urdf.xacro"/>

File: urdf/sample_holder_system.xacro (robot description, xacro)
@@ -16,18 +16,18 @@
             <parent link="centre_rot_stage_link"/>
             <child link="sample_link"/>
-            <origin xyz="0 0.015 0.00" rpy="0 0.0 0.0"/>
+            <origin xyz="0 0.015 0.00" rpy="-${pi/2} 0.0 0.0"/>
         </joint>
         <link name="sample_link">
             <visual>
-                <origin rpy="0 0 0" xyz="0 -0.0075 0"/>
+                <origin rpy="0 0 0" xyz="0 0 -0.0075"/>
                 <geometry>
-                    <box size="0.03 0.015 0.03"/>
+                    <box size="0.03 0.03 0.015"/>
                 </geometry>
                 <material name="orange"/>
             </visual>
                 <collision>
-                <origin rpy="0 0 0" xyz="0 -0.0075 0"/>
+                <origin rpy="0 0 0" xyz="0 0 -0.0075 "/>
                 <geometry>
-                    <box size="0.03 0.015 0.03"/>
+                    <box size="0.03 0.03 0.015"/>
                 </geometry>
             </collision>

File: urdf/samples/brain_slice.urdf.xacro (robot description, xacro)
@@ -9,5 +9,5 @@
         </inertial>
         <visual>
-        <origin rpy="${-pi/2} 0 0" xyz="0 0 0"/>
+        <origin rpy="0 0 0" xyz="0 0 0"/>
         <geometry>
             <mesh filename="package://micro_resector_description/meshes/samples/brain_slice.stl" scale="0.002 0.002 0.002"/>
@@ -16,5 +16,5 @@
         </visual>
         <collision>
-        <origin rpy="${-pi/2} 0 0" xyz="0 0 0"/>
+        <origin rpy="0 0 0" xyz="0 0 0"/>
         <geometry>
             <mesh filename="package://micro_resector_description/meshes/samples/brain_slice.stl" scale="0.002 0.002 0.002"/>

File: urdf/tools/scalpel.xacro (robot description, xacro)
@@ -22,9 +22,15 @@
     </collision>
   </link>
-  <link name="${prefix}_scalpel_blade_link"/>
+  <link name="${prefix}_scalpel_blade_base_link"/>
   <joint name="${prefix}_scalpel_joint" type="fixed">
-    <origin rpy="-${pi/2} 0 0" xyz="-0.013757 0.008025 -0.152227"/>
+    <origin rpy="0 ${pi/2} 0" xyz="-0.013757 0.008025 -0.152227"/>
     <parent link="${prefix}_scalpel_base_link"/>
-    <child link="${prefix}_scalpel_blade_link"/>
+    <child link="${prefix}_scalpel_blade_base_link"/>
+  </joint>
+  <link name="${prefix}_scalpel_blade_tip_link"/>
+  <joint name="${prefix}_scalpel_blade_joint" type="fixed">
+    <origin rpy="0 0 0" xyz="0.002 0 0"/>
+    <parent link="${prefix}_scalpel_blade_base_link"/>
+    <child link="${prefix}_scalpel_blade_tip_link"/>
   </joint>
 </xacro:macro>

Commit message: Scalpel updated to new tool and docker file made for the repo

File: urdf/full_setup.urdf.xacro (robot description, xacro)
@@ -5,9 +5,9 @@
     <link name="base_link"/>
     <xacro:include filename="$(find micro_resector_description)/urdf/materials.xacro" />
-    <xacro:include filename="$(find micro_resector_description)/urdf/tweezer_system.xacro" />
+    <!-- <xacro:include filename="$(find micro_resector_description)/urdf/tweezer_system.xacro" /> -->
     <xacro:include filename="$(find micro_resector_description)/urdf/scalpel_system.xacro"/>
     <xacro:include filename="$(find micro_resector_description)/urdf/sample_holder_system.xacro"/>
     <xacro:include filename="$(find micro_resector_description)/urdf/tools/microscope_camera.xacro"/>
-    <joint name="tweezer_to_base" type="fixed">
+    <!-- <joint name="tweezer_to_base" type="fixed">
         <parent link="base_link"/>
         <child link="tweezer_system_base_link"/>
@@ -15,9 +15,9 @@
     </joint>
     <xacro:tweezer_system hardware_interface="$(arg hardware_interface)">
-    </xacro:tweezer_system>
+    </xacro:tweezer_system> -->
     <joint name="scalpel_to_base" type="fixed">
         <parent link="base_link"/>
         <child link="scalpel_system_base_link"/>
-        <origin xyz="-0.15 -0.042525 0.00" rpy="0.0 0.0 0.0"/>
+        <origin xyz="-0.0990 -0.037525 0.005" rpy="0.0 0.0 0.0"/>
     </joint>
     <xacro:scalpel_system hardware_interface="$(arg hardware_interface)">

File: urdf/tools/scalpel.xacro (robot description, xacro)
@@ -9,14 +9,14 @@
     </inertial>
     <visual>
-      <origin rpy="-${pi/2} -${pi/2} 0" xyz="-0.0375 -0.0345 0.0"/>
+      <origin rpy="${pi} -${pi/2} 0" xyz="0 0 0"/>
       <geometry>
-        <mesh filename="package://micro_resector_description/meshes/tools/scalpel.stl" scale="0.001 0.001 0.001"/>
+        <mesh filename="package://micro_resector_description/meshes/tools/scalpel_assembly.stl"/>
       </geometry>
       <material name="blue"/>
     </visual>
     <collision>
-      <origin rpy="-${pi/2} -${pi/2} 0" xyz="-0.0375 -0.0345 0.0"/>
+      <origin rpy="${pi} -${pi/2} 0" xyz="0 0 0"/>
       <geometry>
-        <mesh filename="package://micro_resector_description/meshes/tools/scalpel.stl" scale="0.001 0.001 0.001"/>
+        <mesh filename="package://micro_resector_description/meshes/tools/scalpel_assembly.stl"/>
       </geometry>
     </collision>
@@ -24,5 +24,5 @@
   <link name="${prefix}_scalpel_blade_base_link"/>
   <joint name="${prefix}_scalpel_joint" type="fixed">
-    <origin rpy="0 ${pi/2} 0" xyz="-0.013757 0.008025 -0.152227"/>
+    <origin rpy="0 ${pi/2} 0" xyz="-0.016431 0.003 -0.089528"/>
     <parent link="${prefix}_scalpel_base_link"/>
     <child link="${prefix}_scalpel_blade_base_link"/>
@@ -30,5 +30,5 @@
   <link name="${prefix}_scalpel_blade_tip_link"/>
   <joint name="${prefix}_scalpel_blade_joint" type="fixed">
-    <origin rpy="0 0 0" xyz="0.0025 0 0"/>
+    <origin rpy="0 0 0" xyz="0.008 0 0"/>
     <parent link="${prefix}_scalpel_blade_base_link"/>
     <child link="${prefix}_scalpel_blade_tip_link"/>
