Commit message: updated tool models and added sample holder models into scene with calibrations

File: urdf/full_setup.urdf.xacro (robot description, xacro)
@@ -5,19 +5,19 @@
     <link name="base_link"/>
     <xacro:include filename="$(find micro_resector_description)/urdf/materials.xacro" />
-    <!-- <xacro:include filename="$(find micro_resector_description)/urdf/tweezer_system.xacro" /> -->
+    <xacro:include filename="$(find micro_resector_description)/urdf/tweezer_system.xacro" />
     <xacro:include filename="$(find micro_resector_description)/urdf/scalpel_system.xacro"/>
     <xacro:include filename="$(find micro_resector_description)/urdf/sample_holder_system.xacro"/>
     <xacro:include filename="$(find micro_resector_description)/urdf/tools/microscope_camera.xacro"/>
-    <!-- <joint name="tweezer_to_base" type="fixed">
+    <joint name="tweezer_to_base" type="fixed">
         <parent link="base_link"/>
         <child link="tweezer_system_base_link"/>
-        <origin xyz="0.15 0.0 0.00" rpy="0 0.0 ${pi}"/>
+        <origin xyz="0.0990 -0.037525 0.00" rpy="0 0.0 0"/>
     </joint>
     <xacro:tweezer_system hardware_interface="$(arg hardware_interface)">
-    </xacro:tweezer_system> -->
+    </xacro:tweezer_system>
     <joint name="scalpel_to_base" type="fixed">
         <parent link="base_link"/>
         <child link="scalpel_system_base_link"/>
-        <origin xyz="-0.0990 -0.037525 0.005" rpy="0.0 0.0 0.0"/>
+        <origin xyz="-0.0990 -0.037525 0.00" rpy="0.0 0.0 0.0"/>
     </joint>
     <xacro:scalpel_system hardware_interface="$(arg hardware_interface)">

File: urdf/sample_holder_system.xacro (robot description, xacro)
@@ -16,18 +16,17 @@
             <parent link="centre_rot_stage_link"/>
             <child link="sample_link"/>
-            <origin xyz="0 0.015 0.00" rpy="-${pi/2} 0.0 0.0"/>
+            <origin xyz="0 0.0101 0.00" rpy="-${pi/2} 0.0 0.0"/>
         </joint>
         <link name="sample_link">
             <visual>
-                <origin rpy="0 0 0" xyz="0 0 -0.0075"/>
+                <origin rpy="0 0 0" xyz="0 0 -0.0101"/>
                 <geometry>
-                    <box size="0.03 0.03 0.015"/>
+                    <mesh filename="package://micro_resector_description/meshes/tools/rotation_base_mount.dae"/>
                 </geometry>
-                <material name="orange"/>
             </visual>
                 <collision>
-                <origin rpy="0 0 0" xyz="0 0 -0.0075 "/>
+                <origin rpy="0 0 0" xyz="0 0 -0.0101"/>
                 <geometry>
-                    <box size="0.03 0.03 0.015"/>
+                     <mesh filename="package://micro_resector_description/meshes/tools/rotation_base_mount.stl"/>
                 </geometry>
             </collision>

File: urdf/tools/tweezer.xacro (robot description, xacro)
@@ -1,60 +1,42 @@
 <?xml version="1.0" ?>
 <robot name="tweezer" xmlns:xacro="http://www.ros.org/wiki/xacro">
-<xacro:macro name="tweezer" params="prefix direction">
-  <xacro:property name="type" value="${direction}"/>
-  <xacro:if value="${type == 'left'}">
-    <link name="${prefix}_tweezer_base_link">
-      <visual>
-        <origin rpy="0 0 -${pi/2}" xyz="-0.133 0.01 0.0"/>
-        <geometry>
-          <mesh filename="package://micro_resector_description/meshes/tools/tweezer_left.stl" scale="0.001 0.001 0.001"/>
-        </geometry>
-        <material name="red"/>
-      </visual>
-      <collision>
-        <origin rpy="0 0 -${pi/2}" xyz="-0.133 0.01 0.0"/>
-        <geometry>
-          <mesh filename="package://micro_resector_description/meshes/tools/tweezer_left.stl" scale="0.001 0.001 0.001"/>
-        </geometry>
-      </collision>
-      <inertial>
-        <mass value="0.1" />
-        <inertia ixx="0.03" iyy="0.03" izz="0.03" ixy="0.0" ixz="0.0" iyz="0.0" />
-      </inertial>
-    </link>
-    <link name="${prefix}_tweezer_prong_link"/>
-    <joint name="${prefix}_tweezer_joint" type="fixed">
-      <origin rpy="${pi} -${pi/2} 0" xyz="-0.015639 0.008 0.15847"/>
-      <parent link="${prefix}_tweezer_base_link"/>
-      <child link="${prefix}_tweezer_prong_link"/>
-    </joint>
-  </xacro:if>
-  <xacro:if value="${type == 'right'}">
-    <link name="${prefix}_tweezer_base_link">
-      <visual>
-        <origin rpy="${pi} 0 ${pi/2}" xyz="-0.133 0.048 0.0"/>
-        <geometry>
-          <mesh filename="package://micro_resector_description/meshes/tools/tweezer_right.stl" scale="0.001 0.001 0.001"/>
-        </geometry>
-        <material name="green"/>
-      </visual>
-      <collision>
-        <origin rpy="${pi} 0 ${pi/2}" xyz="-0.133 0.048 0.0"/>
-        <geometry>
-          <mesh filename="package://micro_resector_description/meshes/tools/tweezer_right.stl" scale="0.001 0.001 0.001"/>
-        </geometry>
-      </collision>
-      <inertial>
-        <mass value="0.1" />
-        <inertia ixx="0.03" iyy="0.03" izz="0.03" ixy="0.0" ixz="0.0" iyz="0.0" />
-      </inertial>
-    </link>
-    <link name="${prefix}_tweezer_prong_link"/>
-    <joint name="${prefix}_tweezer_joint" type="fixed">
-      <origin rpy="0 ${pi/2} 0" xyz="-0.015639 0.008 -0.15847"/>
-      <parent link="${prefix}_tweezer_base_link"/>
-      <child link="${prefix}_tweezer_prong_link"/>
-    </joint>
-  </xacro:if>
+<xacro:macro name="tweezer" params="prefix">
+  <link name="${prefix}_tweezer_base_link">
+    <inertial>
+      <origin rpy="${pi/2} -${pi/2} 0" xyz="0.0 0.0075 0.0"/>
+      <mass value="0.058579061972031825"/>
+      <inertia ixx="1.2e-05" ixy="-0.0" ixz="-0.0" iyy="2.4e-05" iyz="0.0" izz="1.2e-05"/>
+    </inertial>
+    <visual>
+      <origin rpy="${pi} ${pi/2} ${pi}" xyz="0 0.006 0"/>
+      <geometry>
+        <mesh filename="package://micro_resector_description/meshes/tools/tweezer_assembly.dae"/>
+      </geometry>
+    </visual>
+    <collision>
+      <origin rpy="${pi} ${pi/2} ${pi}" xyz="0 0.006 0"/>
+      <geometry>
+        <mesh filename="package://micro_resector_description/meshes/tools/tweezer_assembly.stl"/>
+      </geometry>
+    </collision>
+  </link>
+  <link name="${prefix}_tweezer_prong_centre_link"/>
+  <joint name="${prefix}_tweezer_joint" type="fixed">
+    <origin rpy="0 -${pi/2} -${pi}" xyz="-0.016482 0.003 0.095201"/> <!--model->urdf x->-z, y->y, z->-x -->
+    <parent link="${prefix}_tweezer_base_link"/>
+    <child link="${prefix}_tweezer_prong_centre_link"/>
+  </joint>
+  <link name="${prefix}_tweezer_left_prong_tip_link"/>
+  <joint name="${prefix}_tweezer_left_prong_tip_joint" type="fixed">
+    <origin rpy="0 0 0" xyz="0.003826 0.00035 0"/>
+    <parent link="${prefix}_tweezer_prong_centre_link"/>
+    <child link="${prefix}_tweezer_left_prong_tip_link"/>
+  </joint>
+  <link name="${prefix}_tweezer_right_prong_tip_link"/>
+  <joint name="${prefix}_tweezer_right_prong_tip_joint" type="fixed">
+    <origin rpy="0 0 0" xyz="0.003826 -0.00035 0"/>
+    <parent link="${prefix}_tweezer_prong_centre_link"/>
+    <child link="${prefix}_tweezer_right_prong_tip_link"/>
+  </joint>
 </xacro:macro>
 </robot>

File: urdf/tweezer_system.xacro (robot description, xacro)
@@ -3,5 +3,4 @@
     <xacro:include filename="$(find micro_resector_description)/urdf/stage/linear_stage.xacro"/>
     <xacro:include filename="$(find micro_resector_description)/urdf/link/l_bracket.xacro"/>
-    <xacro:include filename="$(find micro_resector_description)/urdf/link/tweezer_spacing_base.xacro"/>
     <xacro:include filename="$(find micro_resector_description)/urdf/tools/tweezer.xacro"/>
     <xacro:macro name="tweezer_system" params="hardware_interface">
@@ -16,68 +15,31 @@
         <xacro:linear_stage hardware_interface="$(arg hardware_interface)" prefix="tweezer_x">
         </xacro:linear_stage>
-        <joint name="tweezer_spacing_stage_joint" type="fixed">
+        <joint name="tweezer_y_linear_stage_joint" type="fixed">
             <parent link="tweezer_x_lin_stage_link"/>
-            <child link="tweezer_spacing_base_link"/>
+            <child link="tweezer_y_lin_base_link"/>
             <origin xyz="0.0 0.0 0.00" rpy="0.0 ${pi/2} 0.0"/>
         </joint>
-        <xacro:tweezer_spacing_base prefix="tweezer">
-        </xacro:tweezer_spacing_base>
-        Left Tweezzer
-        <joint name="tweezer_left_stage_spacing_bracket_joint" type="fixed">
-            <parent link="tweezer_spacing_left_side_link"/>
-            <child link="tweezer_left_y_lin_base_link"/>
+        <xacro:linear_stage hardware_interface="$(arg hardware_interface)" prefix="tweezer_y">
+        </xacro:linear_stage>
+        <joint name="tweezer_l_bracket_joint" type="fixed">
+            <parent link="tweezer_y_lin_stage_link"/>
+            <child link="tweezer_z_bracket_base_link"/>
+            <origin xyz="0.0 0.0 0.00" rpy="0.0 ${pi/2} 0.0"/>
+        </joint>
+        <xacro:l_bracket prefix="tweezer_z">
+        </xacro:l_bracket>
+        <joint name="tweezer_z_linear_stage_joint" type="fixed">
+            <parent link="tweezer_z_bracket_side_link"/>
+            <child link="tweezer_z_lin_base_link"/>
+            <origin xyz="0.0 0.0 0.00" rpy="0.0 ${pi/2} 0.0"/>
+        </joint>
+        <xacro:linear_stage hardware_interface="$(arg hardware_interface)" prefix="tweezer_z">
+        </xacro:linear_stage>
+        <joint name="tweezer_joint" type="fixed">
+            <parent link="tweezer_z_lin_stage_link"/>
+            <child link="tweezer_z_tweezer_base_link"/>
             <origin xyz="0.0 0.0 0.00" rpy="0.0 0.0 0.0"/>
         </joint>
-        <xacro:linear_stage hardware_interface="$(arg hardware_interface)" prefix="tweezer_left_y">
-        </xacro:linear_stage>
-        <joint name="tweezer_left_l_bracket_joint" type="fixed">
-            <parent link="tweezer_left_y_lin_stage_link"/>
-            <child link="tweezer_left_z_bracket_base_link"/>
-            <origin xyz="0.0 0.0 0.00" rpy="0.0 -${pi/2} 0.0"/>
-        </joint>
-        <xacro:l_bracket prefix="tweezer_left_z">
-        </xacro:l_bracket>
-        <joint name="tweezer_left_z_linear_stage_joint" type="fixed">
-            <parent link="tweezer_left_z_bracket_side_link"/>
-            <child link="tweezer_left_z_lin_base_link"/>
-            <origin xyz="0.0 0.0 0.00" rpy="0.0 ${pi/2} 0.0"/>
-        </joint>
-        <xacro:linear_stage hardware_interface="$(arg hardware_interface)" prefix="tweezer_left_z">
-        </xacro:linear_stage>
-        <joint name="tweezer_left_joint" type="fixed">
-            <parent link="tweezer_left_z_lin_stage_link"/>
-            <child link="left_tweezer_base_link"/>
-            <origin xyz="0.0 0.0 0.00" rpy="0.0 0.0 0.0"/>
-        </joint>
-        <xacro:tweezer prefix="left" direction="left">
-        </xacro:tweezer>
-        <!-- Right Tweezzer -->
-        <joint name="tweezer_right_stage_spacing_bracket_joint" type="fixed">
-            <parent link="tweezer_spacing_right_side_link"/>
-            <child link="tweezer_right_y_lin_base_link"/>
-            <origin xyz="0.0 0.0 0.00" rpy="0.0 0.0 0.0"/>
-        </joint>
-        <xacro:linear_stage hardware_interface="$(arg hardware_interface)" prefix="tweezer_right_y">
-        </xacro:linear_stage>
-        <joint name="tweezer_right_l_bracket_joint" type="fixed">
-            <parent link="tweezer_right_y_lin_stage_link"/>
-            <child link="tweezer_right_z_bracket_base_link"/>
-            <origin xyz="0.0 0.0 0.00" rpy="0.0 ${pi/2} 0.0"/>
-        </joint>
-        <xacro:l_bracket prefix="tweezer_right_z">
-        </xacro:l_bracket>
-        <joint name="tweezer_right_z_linear_stage_joint" type="fixed">
-            <parent link="tweezer_right_z_bracket_side_link"/>
-            <child link="tweezer_right_z_lin_base_link"/>
-            <origin xyz="0.0 0.0 0.00" rpy="0.0 ${pi/2} 0.0"/>
-        </joint>
-        <xacro:linear_stage hardware_interface="$(arg hardware_interface)" prefix="tweezer_right_z">
-        </xacro:linear_stage>
-        <joint name="tweezer_right_joint" type="fixed">
-            <parent link="tweezer_right_z_lin_stage_link"/>
-            <child link="right_tweezer_base_link"/>
-            <origin xyz="0.0 0.0 0.00" rpy="0.0 0.0 0.0"/>
-        </joint>
-        <xacro:tweezer prefix="right" direction="right">
+        <xacro:tweezer prefix="tweezer_z">
         </xacro:tweezer>
     </xacro:macro>

Commit message: tool updated

File: urdf/full_setup.urdf.xacro (robot description, xacro)
@@ -1,4 +1,4 @@
 <?xml version="1.0"?>
-<robot xmlns:xacro="http://www.ros.org/wiki/xacro" name="stage">
+<robot xmlns:xacro="http://www.ros.org/wiki/xacro" name="micro_resector">
     <xacro:arg name="hardware_interface" default="PositionJointInterface"/>
     <xacro:arg name="prefix" default="x"/>

File: urdf/tools/microscope_camera.xacro (robot description, xacro)
@@ -10,5 +10,5 @@
                 <origin xyz="${-camera_dim/2} 0 0 " rpy="0 ${-pi/2} 0"/>
                 <geometry>
-                    <cylinder radius="${-camera_dim/2}" length="${camera_dim}"/>
+                    <cylinder radius="${camera_dim/2}" length="${camera_dim}"/>
                 </geometry>
             </collision>
@@ -16,5 +16,5 @@
                 <origin xyz="${-camera_dim/2} 0 0" rpy="0 ${-pi/2} 0"/>
                 <geometry>
-                    <cylinder radius="${-camera_dim/2}" length="${camera_dim}"/>
+                    <cylinder radius="${camera_dim/2}" length="${camera_dim}"/>
                 </geometry>
                 <material name="red"/>
