Commit message: Rewrote xacro files for setup, updated linear stage meshes, split tools to tool holder and actual attachment

File: urdf/full_setup.urdf.xacro (robot description, xacro)
@@ -3,4 +3,6 @@
     <xacro:arg name="hardware_interface" default="PositionJointInterface"/>
     <xacro:arg name="prefix" default="x"/>
+    <xacro:arg name="virtual_joints" default="false"/>
+    <xacro:arg name="camera" default="true"/>
     <link name="base_link"/>
     <xacro:include filename="$(find micro_resector_description)/urdf/materials.xacro" />
@@ -9,31 +11,61 @@
     <xacro:include filename="$(find micro_resector_description)/urdf/sample_holder_system.xacro"/>
     <xacro:include filename="$(find micro_resector_description)/urdf/tools/microscope_camera.xacro"/>
-    <joint name="tweezer_to_base" type="fixed">
-        <parent link="base_link"/>
-        <child link="tweezer_system_base_link"/>
-        <origin xyz="0.0990 -0.037525 0.00" rpy="0 0.0 0"/>
-    </joint>
-    <xacro:tweezer_system hardware_interface="$(arg hardware_interface)">
+    <xacro:if value="$(arg virtual_joints)">
+        <joint name="tweezer_to_base" type="floating">
+            <parent link="base_link"/>
+            <child link="tweezer_system_base_link"/>
+            <origin xyz="0.0990 -0.037525 0.00" rpy="0 0.0 0"/>
+        </joint>
+        <joint name="scalpel_to_base" type="floating">
+            <parent link="base_link"/>
+            <child link="scalpel_system_base_link"/>
+            <origin xyz="-0.0990 -0.037525 0.00" rpy="0.0 0.0 ${pi/2}"/>
+        </joint>
+        <joint name="sample_holder_to_base" type="floating">
+            <parent link="base_link"/>
+            <child link="sample_holder_base_link"/>
+            <origin xyz="0 0 0.00" rpy="0 0.0 0.0"/>
+        </joint>
+        <xacro:if value="$(arg camera)">
+            <joint name="camera_joint" type="floating">
+                <origin xyz="0 0 0.1" rpy="0 ${pi/2} 0"/>
+                <parent link="base_link"/>
+                <child link="camera_link"/>
+            </joint>
+        </xacro:if>
+    </xacro:if>
+    <xacro:unless value="$(arg virtual_joints)">
+        <joint name="tweezer_to_base" type="fixed">
+            <parent link="base_link"/>
+            <child link="tweezer_system_base_link"/>
+            <origin xyz="0.0990 -0.037525 0.00" rpy="0 0.0 ${pi}"/>
+        </joint>
+        <joint name="scalpel_to_base" type="fixed">
+            <parent link="base_link"/>
+            <child link="scalpel_system_base_link"/>
+            <origin xyz="-0.0990 -0.037525 0.00" rpy="0.0 0.0 0"/>
+        </joint>
+        <joint name="sample_holder_to_base" type="fixed">
+            <parent link="base_link"/>
+            <child link="sample_holder_base_link"/>
+            <origin xyz="0 0 0.00" rpy="0 0.0 0.0"/>
+        </joint>
+        <xacro:if value="$(arg camera)">
+            <joint name="camera_joint" type="fixed">
+                <origin xyz="0 0 0.1" rpy="0 ${pi/2} 0"/>
+                <parent link="base_link"/>
+                <child link="camera_link"/>
+            </joint>
+        </xacro:if>
+    </xacro:unless>
+    <xacro:tweezer_system hardware_interface="$(arg hardware_interface)" name="tweezer">
     </xacro:tweezer_system>
-    <joint name="scalpel_to_base" type="fixed">
-        <parent link="base_link"/>
-        <child link="scalpel_system_base_link"/>
-        <origin xyz="-0.0990 -0.037525 0.00" rpy="0.0 0.0 0.0"/>
-    </joint>
-    <xacro:scalpel_system hardware_interface="$(arg hardware_interface)">
+    <xacro:scalpel_system hardware_interface="$(arg hardware_interface)" name="scalpel">
     </xacro:scalpel_system>
-    <joint name="sample_holder_to_base" type="fixed">
-        <parent link="base_link"/>
-        <child link="sample_holder_base_link"/>
-        <origin xyz="0 0 0.00" rpy="0 0.0 0.0"/>
-    </joint>
     <xacro:sample_holder hardware_interface="$(arg hardware_interface)">
     </xacro:sample_holder>
-    <joint name="camera_joint" type="fixed">
-        <origin xyz="0 0 0.1" rpy="0 ${pi/2} 0"/>
-        <parent link="base_link"/>
-        <child link="camera_link"/>
-    </joint>
-    <xacro:microscope_camera type="mono"/>
+    <xacro:if value="$(arg camera)">
+        <xacro:microscope_camera type="mono"/>
+    </xacro:if>
     <joint name="sample_joint" type="fixed">
         <parent link="sample_link"/>

File: urdf/link/l_bracket.xacro (robot description, xacro)
@@ -9,14 +9,13 @@
     </inertial>
     <visual>
-      <origin rpy="0 0 0" xyz="0 -0.01 0"/>
+      <origin rpy="0 0 0" xyz="0 0 0"/>
       <geometry>
-        <mesh filename="package://micro_resector_description/meshes/link/l_bracket.stl" scale="0.001 0.001 0.001"/>
+        <mesh filename="package://micro_resector_description/meshes/link/l_bracket.dae"/>
       </geometry>
-      <material name="silver"/>
     </visual>
     <collision>
-      <origin rpy="0 0 0" xyz="0 -0.01 0"/>
+      <origin rpy="0 0 0" xyz="0 0 0"/>
       <geometry>
-        <mesh filename="package://micro_resector_description/meshes/link/l_bracket.stl" scale="0.001 0.001 0.001"/>
+        <mesh filename="package://micro_resector_description/meshes/link/l_bracket.stl"/>
       </geometry>
     </collision>
@@ -24,5 +23,5 @@
   <link name="${prefix}_bracket_side_link"/>
   <joint name="${prefix}_bracket_joint" type="fixed">
-    <origin rpy="${pi/2} 0 0" xyz="0.0 0.028 0.025"/>
+    <origin rpy="${pi/2} 0 0" xyz="0.0 -0.025 0.03"/>
     <parent link="${prefix}_bracket_base_link"/>
     <child link="${prefix}_bracket_side_link"/>

File: urdf/scalpel_system.xacro (robot description, xacro)
@@ -1,41 +1,50 @@
 <?xml version="1.0"?>
-<robot xmlns:xacro="http://www.ros.org/wiki/xacro" name="scalpel_system">
+<robot xmlns:xacro="http://www.ros.org/wiki/xacro">
     <xacro:include filename="$(find micro_resector_description)/urdf/stage/linear_stage.xacro"/>
     <xacro:include filename="$(find micro_resector_description)/urdf/link/l_bracket.xacro"/>
     <xacro:include filename="$(find micro_resector_description)/urdf/tools/scalpel.xacro"/>
-    <xacro:macro name="scalpel_system" params="hardware_interface">
-        <xacro:arg name="hardware_interface" default="PositionJointInterface"/>
-        <xacro:arg name="prefix" default="x"/>
-        <link name="scalpel_system_base_link"/>
-        <joint name="scalpel_x_linear_stage_world_joint" type="fixed">
-            <parent link="scalpel_system_base_link"/>
-            <child link="scalpel_x_lin_base_link"/>
-            <origin xyz="0.0 0.0 0.00" rpy="${pi/2} 0.0 0.0"/>
+    <xacro:include filename="$(find micro_resector_description)/urdf/tools/tool_holder.xacro"/>
+    <xacro:macro name="scalpel_system" params="hardware_interface name">
+<!--        <xacro:arg name="hardware_interface" default="PositionJointInterface"/>-->
+<!--        <xacro:arg name="name" default="scalpel"/>-->
+        <link name="${name}_system_base_link"/>
+        <joint name="${name}_x_linear_stage_world_joint" type="fixed">
+            <parent link="${name}_system_base_link"/>
+            <child link="${name}_x_lin_base_link"/>
+            <origin xyz="0 0 0" rpy="0 0 0"/>
         </joint>
-        <xacro:linear_stage hardware_interface="$(arg hardware_interface)" prefix="scalpel_x">
+        <xacro:linear_stage hardware_interface="${hardware_interface}" prefix="${name}_x">
         </xacro:linear_stage>
-        <joint name="scalpel_y_linear_stage_joint" type="fixed">
-            <parent link="scalpel_x_lin_stage_link"/>
-            <child link="scalpel_y_lin_base_link"/>
-            <origin xyz="0.0 0.0 0.00" rpy="0.0 ${pi/2} 0.0"/>
+        <joint name="${name}_y_linear_stage_joint" type="fixed">
+            <parent link="${name}_x_lin_stage_link"/>
+            <child link="${name}_y_lin_base_link"/>
+            <origin xyz="0 0 0" rpy="0 0 ${pi/2}"/>
+<!--            <origin xyz="0.0 0.0 0.00" rpy="0.0 0.0 ${pi/2}"/>-->
         </joint>
-        <xacro:linear_stage hardware_interface="$(arg hardware_interface)" prefix="scalpel_y">
+        <xacro:linear_stage hardware_interface="${hardware_interface}" prefix="${name}_y">
         </xacro:linear_stage>
-        <joint name="scalpel_l_bracket_joint" type="fixed">
-            <parent link="scalpel_y_lin_stage_link"/>
-            <child link="scalpel_z_bracket_base_link"/>
-            <origin xyz="0.0 0.0 0.00" rpy="0.0 ${pi/2} 0.0"/>
+        <joint name="${name}_l_bracket_joint" type="fixed">
+            <parent link="${name}_y_lin_stage_link"/>
+            <child link="${name}_z_bracket_base_link"/>
+            <origin xyz="0.0 0.0 0.00" rpy="0.0 0 ${pi/2}"/>
         </joint>
-        <xacro:l_bracket prefix="scalpel_z">
+        <xacro:l_bracket prefix="${name}_z">
         </xacro:l_bracket>
-        <joint name="scalpel_z_linear_stage_joint" type="fixed">
-            <parent link="scalpel_z_bracket_side_link"/>
-            <child link="scalpel_z_lin_base_link"/>
-            <origin xyz="0.0 0.0 0.00" rpy="0.0 ${pi/2} 0.0"/>
+        <joint name="${name}_z_linear_stage_joint" type="fixed">
+            <parent link="${name}_z_bracket_side_link"/>
+            <child link="${name}_z_lin_base_link"/>
+            <origin xyz="0.0 0.0 0.00" rpy="0 0 -${pi/2}"/>
         </joint>
-        <xacro:linear_stage hardware_interface="$(arg hardware_interface)" prefix="scalpel_z">
+        <xacro:linear_stage hardware_interface="${hardware_interface}" prefix="${name}_z">
         </xacro:linear_stage>
-        <joint name="scalpel_joint" type="fixed">
-            <parent link="scalpel_z_lin_stage_link"/>
+        <joint name="${name}_tool_holder_joint" type="fixed">-->
+            <parent link="${name}_z_lin_stage_link"/>
+            <child link="${name}_tool_holder_link"/>
+            <origin xyz="0 0 0" rpy="0 0 ${pi/2}"/>
+        </joint>
+        <xacro:tool_holder name="${name}">
+        </xacro:tool_holder>
+        <joint name="${name}_attachment_joint" type="fixed">
+            <parent link="${name}_tool_attachment_link"/>
             <child link="scalpel_z_scalpel_base_link"/>
             <origin xyz="0.0 0.0 0.00" rpy="0.0 0.0 0.0"/>

File: urdf/stage/linear_stage.xacro (robot description, xacro)
@@ -6,19 +6,19 @@
   <link name="${prefix}_lin_base_link">
     <inertial>
-      <origin rpy="0 0 0" xyz="0.0 0.0015 0.0"/>
+      <origin rpy="0 0 0" xyz="0 0 0"/>
       <mass value="0.058579061972031825"/>
       <inertia ixx="1.2e-05" ixy="-0.0" ixz="-0.0" iyy="2.4e-05" iyz="0.0" izz="1.2e-05"/>
     </inertial>
     <visual>
-      <origin rpy="0 0 0" xyz="0 0.0095 0"/>
+      <origin rpy="0 0 0" xyz="0 0 0"/>
       <geometry>
-        <mesh filename="package://micro_resector_description/meshes/stage/lin_base_link.stl" scale="0.001 0.001 0.001"/>
+        <mesh filename="package://micro_resector_description/meshes/stage/lin_base_link.dae"/>
       </geometry>
       <material name="silver"/>
     </visual>
     <collision>
-      <origin rpy="0 0 0" xyz="0 0.0095 0"/>
+      <origin rpy="0 0 0" xyz="0 0 0"/>
       <geometry>
-        <mesh filename="package://micro_resector_description/meshes/stage/lin_base_link.stl" scale="0.001 0.001 0.001"/>
+        <mesh filename="package://micro_resector_description/meshes/stage/lin_base_link.stl"/>
       </geometry>
     </collision>
@@ -26,24 +26,24 @@
   <link name="${prefix}_lin_stage_link">
     <inertial>
-      <origin rpy="0 0 0" xyz="0.0 -0.00028 0.0"/>
+      <origin rpy="0 0 0" xyz="0 0 0"/>
       <mass value="0.11339718225370693"/>
       <inertia ixx="2.3e-05" ixy="0.0" ixz="0.0" iyy="4.6e-05" iyz="0.0" izz="2.3e-05"/>
     </inertial>
     <visual>
-      <origin rpy="0 0 0" xyz="0.0 0.0 -0.0"/>
+      <origin rpy="0 0 0" xyz="0 0 0"/>
       <geometry>
-        <mesh filename="package://micro_resector_description/meshes/stage/lin_stage_link.stl" scale="0.001 0.001 0.001"/>
+        <mesh filename="package://micro_resector_description/meshes/stage/lin_stage_link.dae"/>
       </geometry>
       <material name="silver"/>
     </visual>
     <collision>
-      <origin rpy="0 0 0" xyz="0.0 0.0 -0.0"/>
+      <origin rpy="0 0 0" xyz="0 0 0"/>
       <geometry>
-        <mesh filename="package://micro_resector_description/meshes/stage/lin_stage_link.stl" scale="0.001 0.001 0.001"/>
+        <mesh filename="package://micro_resector_description/meshes/stage/lin_stage_link.stl"/>
       </geometry>
     </collision>
   </link>
   <joint name="${prefix}_lin_joint" type="prismatic">
-    <origin rpy="0 0 0" xyz="0.0 0.0095 0.0"/>
+    <origin rpy="0 0 0" xyz="0 0 0.00965"/>
     <parent link="${prefix}_lin_base_link"/>
     <child link="${prefix}_lin_stage_link"/>

File: urdf/tools/scalpel.xacro (robot description, xacro)
@@ -4,19 +4,18 @@
   <link name="${prefix}_scalpel_base_link">
     <inertial>
-      <origin rpy="-${pi/2} -${pi/2} 0" xyz="0.0 0.0075 0.0"/>
+      <origin rpy="0 0 0" xyz="0.0 0.0 0.0"/>
       <mass value="0.058579061972031825"/>
       <inertia ixx="1.2e-05" ixy="-0.0" ixz="-0.0" iyy="2.4e-05" iyz="0.0" izz="1.2e-05"/>
     </inertial>
     <visual>
-      <origin rpy="${pi} -${pi/2} 0" xyz="0 0 0"/>
+      <origin rpy="0 0 0" xyz="0 0 0"/>
       <geometry>
-        <mesh filename="package://micro_resector_description/meshes/tools/scalpel_assembly.stl"/>
+        <mesh filename="package://micro_resector_description/meshes/tools/blade_sm65.dae"/>
       </geometry>
-      <material name="blue"/>
     </visual>
     <collision>
-      <origin rpy="${pi} -${pi/2} 0" xyz="0 0 0"/>
+      <origin rpy="0 0 0" xyz="0 0 0"/>
       <geometry>
-        <mesh filename="package://micro_resector_description/meshes/tools/scalpel_assembly.stl"/>
+        <mesh filename="package://micro_resector_description/meshes/tools/blade_sm65.dae"/>
       </geometry>
     </collision>
@@ -24,5 +23,5 @@
   <link name="${prefix}_scalpel_blade_base_link"/>
   <joint name="${prefix}_scalpel_joint" type="fixed">
-    <origin rpy="0 ${pi/2} 0" xyz="-0.016431 0.003 -0.089528"/>
+    <origin rpy="${-pi/2} 0 ${20.487 * pi/180}" xyz="0.024506 -0.00115 0"/>
     <parent link="${prefix}_scalpel_base_link"/>
     <child link="${prefix}_scalpel_blade_base_link"/>

File: urdf/tools/tweezer.xacro (robot description, xacro)
@@ -9,13 +9,13 @@
     </inertial>
     <visual>
-      <origin rpy="${pi} ${pi/2} ${pi}" xyz="0 0.006 0"/>
+      <origin rpy="0 0 0" xyz="0 0 0"/>
       <geometry>
-        <mesh filename="package://micro_resector_description/meshes/tools/tweezer_assembly.dae"/>
+        <mesh filename="package://micro_resector_description/meshes/tools/tweezer.dae"/>
       </geometry>
     </visual>
     <collision>
-      <origin rpy="${pi} ${pi/2} ${pi}" xyz="0 0.006 0"/>
+      <origin rpy="0 0 0" xyz="0 0 0"/>
       <geometry>
-        <mesh filename="package://micro_resector_description/meshes/tools/tweezer_assembly.stl"/>
+        <mesh filename="package://micro_resector_description/meshes/tools/tweezer.stl"/>
       </geometry>
     </collision>
@@ -23,5 +23,5 @@
   <link name="${prefix}_tweezer_prong_centre_link"/>
   <joint name="${prefix}_tweezer_joint" type="fixed">
-    <origin rpy="0 -${pi/2} -${pi}" xyz="-0.016482 0.003 0.095201"/> <!--model->urdf x->-z, y->y, z->-x -->
+    <origin rpy="${-pi/2} 0 ${21.063 * pi/180}" xyz="0.029821 0.000836 0"/> <!--model->urdf x->-z, y->y, z->-x -->
     <parent link="${prefix}_tweezer_base_link"/>
     <child link="${prefix}_tweezer_prong_centre_link"/>

File: urdf/tweezer_system.xacro (robot description, xacro)
@@ -1,41 +1,50 @@
 <?xml version="1.0"?>
-<robot xmlns:xacro="http://www.ros.org/wiki/xacro" name="tweezer_system">
+<robot xmlns:xacro="http://www.ros.org/wiki/xacro">
     <xacro:include filename="$(find micro_resector_description)/urdf/stage/linear_stage.xacro"/>
     <xacro:include filename="$(find micro_resector_description)/urdf/link/l_bracket.xacro"/>
     <xacro:include filename="$(find micro_resector_description)/urdf/tools/tweezer.xacro"/>
-    <xacro:macro name="tweezer_system" params="hardware_interface">
-        <xacro:arg name="hardware_interface" default="PositionJointInterface"/>
-        <xacro:arg name="prefix" default="x"/>
-        <link name="tweezer_system_base_link"/>
-        <joint name="tweezer_x_linear_stage_world_joint" type="fixed">
-            <parent link="tweezer_system_base_link"/>
-            <child link="tweezer_x_lin_base_link"/>
-            <origin xyz="0.0 0.0 0.00" rpy="${pi/2} 0.0 0.0"/>
+    <xacro:include filename="$(find micro_resector_description)/urdf/tools/tool_holder.xacro"/>
+    <xacro:macro name="tweezer_system" params="hardware_interface name">
+<!--        <xacro:arg name="hardware_interface" default="PositionJointInterface"/>-->
+<!--        <xacro:arg name="name" default="tweezer"/>-->
+        <link name="${name}_system_base_link"/>
+        <joint name="${name}_x_linear_stage_world_joint" type="fixed">
+            <parent link="${name}_system_base_link"/>
+            <child link="${name}_x_lin_base_link"/>
+            <origin xyz="0 0 0" rpy="0 0 0"/>
         </joint>
-        <xacro:linear_stage hardware_interface="$(arg hardware_interface)" prefix="tweezer_x">
+        <xacro:linear_stage hardware_interface="${hardware_interface}" prefix="${name}_x">
         </xacro:linear_stage>
-        <joint name="tweezer_y_linear_stage_joint" type="fixed">
-            <parent link="tweezer_x_lin_stage_link"/>
-            <child link="tweezer_y_lin_base_link"/>
-            <origin xyz="0.0 0.0 0.00" rpy="0.0 ${pi/2} 0.0"/>
+        <joint name="${name}_y_linear_stage_joint" type="fixed">
+            <parent link="${name}_x_lin_stage_link"/>
+            <child link="${name}_y_lin_base_link"/>
+            <origin xyz="0 0 0" rpy="0 0 ${-pi/2}"/>
+<!--            <origin xyz="0.0 0.0 0.00" rpy="0.0 0.0 ${pi/2}"/>-->
         </joint>
-        <xacro:linear_stage hardware_interface="$(arg hardware_interface)" prefix="tweezer_y">
+        <xacro:linear_stage hardware_interface="${hardware_interface}" prefix="${name}_y">
         </xacro:linear_stage>
-        <joint name="tweezer_l_bracket_joint" type="fixed">
-            <parent link="tweezer_y_lin_stage_link"/>
-            <child link="tweezer_z_bracket_base_link"/>
-            <origin xyz="0.0 0.0 0.00" rpy="0.0 ${pi/2} 0.0"/>
+        <joint name="${name}_l_bracket_joint" type="fixed">
+            <parent link="${name}_y_lin_stage_link"/>
+            <child link="${name}_z_bracket_base_link"/>
+            <origin xyz="0.0 0.0 0.0" rpy="0.0 0 ${pi/2}"/>
         </joint>
-        <xacro:l_bracket prefix="tweezer_z">
+        <xacro:l_bracket prefix="${name}_z">
         </xacro:l_bracket>
-        <joint name="tweezer_z_linear_stage_joint" type="fixed">
-            <parent link="tweezer_z_bracket_side_link"/>
-            <child link="tweezer_z_lin_base_link"/>
-            <origin xyz="0.0 0.0 0.00" rpy="0.0 ${pi/2} 0.0"/>
+        <joint name="${name}_z_linear_stage_joint" type="fixed">
+            <parent link="${name}_z_bracket_side_link"/>
+            <child link="${name}_z_lin_base_link"/>
+            <origin xyz="0.0 0.0 0.00" rpy="0 0 -${pi/2}"/>
         </joint>
-        <xacro:linear_stage hardware_interface="$(arg hardware_interface)" prefix="tweezer_z">
+        <xacro:linear_stage hardware_interface="${hardware_interface}" prefix="${name}_z">
         </xacro:linear_stage>
-        <joint name="tweezer_joint" type="fixed">
-            <parent link="tweezer_z_lin_stage_link"/>
+        <joint name="${name}_tool_holder_joint" type="fixed">-->
+            <parent link="${name}_z_lin_stage_link"/>
+            <child link="${name}_tool_holder_link"/>
+            <origin xyz="0 0 0.006" rpy="0 ${pi} ${pi/2}"/>
+        </joint>
+        <xacro:tool_holder name="${name}">
+        </xacro:tool_holder>
+        <joint name="${name}_attachment_joint" type="fixed">
+            <parent link="${name}_tool_attachment_link"/>
             <child link="tweezer_z_tweezer_base_link"/>
             <origin xyz="0.0 0.0 0.00" rpy="0.0 0.0 0.0"/>

Commit message: Set axis of rotation stage to -1 and modified full setup to optical table attachments

File: urdf/full_setup.urdf.xacro (robot description, xacro)
@@ -15,10 +15,10 @@
             <parent link="base_link"/>
             <child link="tweezer_system_base_link"/>
-            <origin xyz="0.0990 -0.037525 0.00" rpy="0 0.0 0"/>
+            <origin xyz="0.098 -0.0375 0.00" rpy="0 0.0 0"/>
         </joint>
         <joint name="scalpel_to_base" type="floating">
             <parent link="base_link"/>
             <child link="scalpel_system_base_link"/>
-            <origin xyz="-0.0990 -0.037525 0.00" rpy="0.0 0.0 ${pi/2}"/>
+            <origin xyz="-0.098 -0.0375 0.00" rpy="0.0 0.0 0"/>
         </joint>
         <joint name="sample_holder_to_base" type="floating">
@@ -39,10 +39,10 @@
             <parent link="base_link"/>
             <child link="tweezer_system_base_link"/>
-            <origin xyz="0.0990 -0.037525 0.00" rpy="0 0.0 ${pi}"/>
+            <origin xyz="0.098 -0.0375 0.00" rpy="0 0 ${pi}"/>
         </joint>
         <joint name="scalpel_to_base" type="fixed">
             <parent link="base_link"/>
             <child link="scalpel_system_base_link"/>
-            <origin xyz="-0.0990 -0.037525 0.00" rpy="0.0 0.0 0"/>
+            <origin xyz="-0.098 -0.0375 0.00" rpy="0.0 0.0 0"/>
         </joint>
         <joint name="sample_holder_to_base" type="fixed">

File: urdf/stage/rotation_stage.xacro (robot description, xacro)
@@ -48,5 +48,5 @@
     <parent link="${prefix}_rot_base_link"/>
     <child link="${prefix}_rot_stage_link"/>
-    <axis xyz="0 1 0.0"/>
+    <axis xyz="0 -1 0.0"/>
     <limit effort="100" velocity="${(pi/180) * 15}"/>
   </joint>
