Commit message: corrected sample holder for new zero procedure

File: urdf/full_setup.urdf.xacro (robot description, xacro)
@@ -73,5 +73,5 @@
         <parent link="sample_link"/>
         <child link="brain_slice_base_link"/>
-        <origin xyz="0 0.0 0.0005" rpy="0 0.0 0.0"/>
+        <origin xyz="0 0.0 0.0005" rpy="0.0 0.0 0"/>
     </joint>
     <xacro:include filename="$(find micro_resector_description)/urdf/samples/brain_slice.urdf.xacro"/>

File: urdf/sample_holder_system.xacro (robot description, xacro)
@@ -16,9 +16,9 @@
             <parent link="centre_rot_stage_link"/>
             <child link="sample_link"/>
-            <origin xyz="0 0.0101 0.00" rpy="-${pi/2} 0.0 0.0"/>
+            <origin xyz="0 0.0101 0.00" rpy="-${pi/2} 0 0.0"/>
         </joint>
         <link name="sample_link">
             <visual>
-                <origin rpy="0 0 0" xyz="0 0 -0.0101"/>
+                <origin rpy="0 0 ${pi/4}" xyz="0 0 -0.0101"/>
                 <geometry>
                     <mesh filename="package://micro_resector_description/meshes/tools/rotation_base_mount.dae"/>
@@ -26,5 +26,5 @@
             </visual>
                 <collision>
-                <origin rpy="0 0 0" xyz="0 0 -0.0101"/>
+                <origin rpy="0 0 ${pi/4}" xyz="0 0 -0.0101"/>
                 <geometry>
                      <mesh filename="package://micro_resector_description/meshes/tools/rotation_base_mount.stl"/>

File: urdf/stage/rotation_stage.xacro (robot description, xacro)
@@ -31,5 +31,5 @@
     </inertial>
     <visual>
-      <origin rpy="0 0 0" xyz="0.0 -0.005 -0.0"/>
+      <origin rpy="0 ${pi/4} 0" xyz="0.0 -0.005 -0.0"/>
       <geometry>
         <mesh filename="package://micro_resector_description/meshes/stage/rot_stage_link.stl" scale="0.001 0.001 0.001"/>
@@ -38,5 +38,5 @@
     </visual>
     <collision>
-      <origin rpy="0 0 0" xyz="0.0 -0.005 -0.0"/>
+      <origin rpy="0 ${pi/4} 0" xyz="0.0 -0.005 -0.0"/>
       <geometry>
         <mesh filename="package://micro_resector_description/meshes/stage/rot_stage_link.stl" scale="0.001 0.001 0.001"/>
@@ -45,5 +45,5 @@
   </link>
   <joint name="${prefix}_rot_joint" type="continuous">
-    <origin rpy="0 ${pi/4} 0" xyz="0.0 0.015 0.0"/>
+    <origin rpy="0 0 0" xyz="0.0 0.015 0.0"/>
     <parent link="${prefix}_rot_base_link"/>
     <child link="${prefix}_rot_stage_link"/>

Commit message: adjusted the sample holder height in the urdf and removed the sample brain slice mesh

File: urdf/full_setup.urdf.xacro (robot description, xacro)
@@ -70,10 +70,10 @@
         <xacro:microscope_camera type="mono"/>
     </xacro:if>
-    <joint name="sample_joint" type="fixed">
-        <parent link="sample_link"/>
-        <child link="brain_slice_base_link"/>
-        <origin xyz="0 0.0 0.0005" rpy="0.0 0.0 0"/>
-    </joint>
-    <xacro:include filename="$(find micro_resector_description)/urdf/samples/brain_slice.urdf.xacro"/>
+<!--    <joint name="sample_joint" type="fixed">-->
+<!--        <parent link="sample_link"/>-->
+<!--        <child link="brain_slice_base_link"/>-->
+<!--        <origin xyz="0 0.0 0.0005" rpy="0.0 0.0 0"/>-->
+<!--    </joint>-->
+<!--    <xacro:include filename="$(find micro_resector_description)/urdf/samples/brain_slice.urdf.xacro"/>-->
     <xacro:include filename="$(find micro_resector_description)/urdf/full_setup.gazebo.xacro"/>
     <xacro:micro_resector_control name="MicroResectorPositionHardwareInterface"

File: urdf/sample_holder_system.xacro (robot description, xacro)
@@ -16,5 +16,5 @@
             <parent link="centre_rot_stage_link"/>
             <child link="sample_link"/>
-            <origin xyz="0 0.0101 0.00" rpy="-${pi/2} 0 0.0"/>
+            <origin xyz="0 0.0085 0.00" rpy="-${pi/2} 0 0.0"/>
         </joint>
         <link name="sample_link">

Commit message: added image sample link frame and calibrated for tweezer offset

File: urdf/full_setup.urdf.xacro (robot description, xacro)
@@ -67,4 +67,10 @@
     <xacro:sample_holder hardware_interface="$(arg hardware_interface)">
     </xacro:sample_holder>
+    <link name="image_sample_link"/>
+    <joint name="image_sample_link_joint" type="fixed">
+        <origin xyz="0 0 0.0235" rpy="0 0 0"/>
+        <parent link="base_link"/>
+        <child link="image_sample_link"/>
+    </joint>
     <xacro:if value="$(arg camera)">
         <xacro:microscope_camera type="mono"/>

File: urdf/tweezer_system.xacro (robot description, xacro)
@@ -43,5 +43,5 @@
             <parent link="${name}_z_lin_stage_link"/>
             <child link="tweezer_tool_holder_link"/>
-            <origin xyz="0 0 0" rpy="${-pi/2} 0 ${pi/2}"/>
+            <origin xyz="0 0.0001 -0.0004" rpy="${-pi/2} 0 ${pi/2}"/>
         </joint>
     </xacro:macro>
