Commit message: tweezer cal adjustment

File: urdf/tweezer_system.xacro (robot description, xacro)
@@ -43,5 +43,5 @@
             <parent link="${name}_z_lin_stage_link"/>
             <child link="tweezer_tool_holder_link"/>
-            <origin xyz="0 0.0001 -0.0004" rpy="${-pi/2} 0 ${pi/2}"/>
+            <origin xyz="0 0.0007 -0.0008" rpy="${-pi/2} 0 ${pi/2}"/>
         </joint>
     </xacro:macro>
