Commit message: Launching with gazebo controllers

File: urdf/link/tweezer_spacing_base.xacro (robot description, xacro)
@@ -16,4 +16,8 @@
       </geometry>
     </collision>
+    <inertial>
+      <mass value="0.1" />
+      <inertia ixx="0.03" iyy="0.03" izz="0.03" ixy="0.0" ixz="0.0" iyz="0.0" />
+    </inertial>
   </link>
   <link name="${prefix}_spacing_left_side_link"/>

File: urdf/materials.xacro (robot description, xacro)
@@ -28,3 +28,6 @@
     <color rgba="1.0 1.0 1.0 1.0"/>
   </material>
+  <gazebo>
+    <plugin filename="libgazebo_ros_control.so" name="control"/>
+  </gazebo>
 </robot>

File: urdf/sample_holder_system.xacro (robot description, xacro)
@@ -32,4 +32,8 @@
                 </geometry>
             </collision>
+            <inertial>
+                <mass value="0.1" />
+                <inertia ixx="0.03" iyy="0.03" izz="0.03" ixy="0.0" ixz="0.0" iyz="0.0" />
+            </inertial>
         </link>
     </xacro:macro>

File: urdf/stage/linear_stage.xacro (robot description, xacro)
@@ -51,6 +51,6 @@
     <limit effort="100" lower="-0.015" upper="0.015" velocity="0.0045"/>
   </joint>
-  <xacro:stage_gazebo prefix="$(arg prefix)" type="lin"/>
-  <xacro:stage_transmission prefix="$(arg prefix)" hardware_interface="${hardware_interface}" type="lin"/>
+  <xacro:stage_gazebo prefix="${prefix}" type="lin"/>
+  <xacro:stage_transmission prefix="${prefix}" hardware_interface="${hardware_interface}" type="lin"/>
 </xacro:macro>
 </robot>

File: urdf/stage/rotation_stage.xacro (robot description, xacro)
@@ -51,6 +51,6 @@
     <limit effort="100" velocity="${(pi/180) * 15}"/>
   </joint>
-  <xacro:stage_gazebo prefix="$(arg prefix)" type="rot"/>
-  <xacro:stage_transmission prefix="$(arg prefix)" hardware_interface="${hardware_interface}" type="rot"/>
+  <xacro:stage_gazebo prefix="${prefix}" type="rot"/>
+  <xacro:stage_transmission prefix="${prefix}" hardware_interface="${hardware_interface}" type="rot"/>
 </xacro:macro>
 </robot>

File: urdf/tools/tweezer.xacro (robot description, xacro)
@@ -18,4 +18,8 @@
         </geometry>
       </collision>
+      <inertial>
+        <mass value="0.1" />
+        <inertia ixx="0.03" iyy="0.03" izz="0.03" ixy="0.0" ixz="0.0" iyz="0.0" />
+      </inertial>
     </link>
     <link name="${prefix}_tweezer_prong_link"/>
@@ -41,4 +45,8 @@
         </geometry>
       </collision>
+      <inertial>
+        <mass value="0.1" />
+        <inertia ixx="0.03" iyy="0.03" izz="0.03" ixy="0.0" ixz="0.0" iyz="0.0" />
+      </inertial>
     </link>
     <link name="${prefix}_tweezer_prong_link"/>

Commit message: modified spacing between the base so the tweezers can be closer to each other, still approximately 4mm offset so will need to redesign the tweezers attachment

File: urdf/link/tweezer_spacing_base.xacro (robot description, xacro)
@@ -23,5 +23,5 @@
   <link name="${prefix}_spacing_left_side_link"/>
   <joint name="${prefix}_spacing_left_joint" type="fixed">
-    <origin rpy="0 0 0" xyz="0.0635 0.005 0"/>
+    <origin rpy="0 0 0" xyz="0.0535 0.005 0"/>
     <parent link="${prefix}_spacing_base_link"/>
     <child link="${prefix}_spacing_left_side_link"/>
@@ -29,5 +29,5 @@
   <link name="${prefix}_spacing_right_side_link"/>
   <joint name="${prefix}_spacing_right_joint" type="fixed">
-    <origin rpy="0 0 0" xyz="-0.0635 0.005 0"/>
+    <origin rpy="0 0 0" xyz="-0.0535 0.005 0"/>
     <parent link="${prefix}_spacing_base_link"/>
     <child link="${prefix}_spacing_right_side_link"/>

File: urdf/tools/scalpel.xacro (robot description, xacro)
@@ -30,5 +30,5 @@
   <link name="${prefix}_scalpel_blade_tip_link"/>
   <joint name="${prefix}_scalpel_blade_joint" type="fixed">
-    <origin rpy="0 0 0" xyz="0.002 0 0"/>
+    <origin rpy="0 0 0" xyz="0.0025 0 0"/>
     <parent link="${prefix}_scalpel_blade_base_link"/>
     <child link="${prefix}_scalpel_blade_tip_link"/>

File: urdf/tools/tweezer.xacro (robot description, xacro)
@@ -25,5 +25,5 @@
     <link name="${prefix}_tweezer_prong_link"/>
     <joint name="${prefix}_tweezer_joint" type="fixed">
-      <origin rpy="${pi/2} 0 0" xyz="-0.015639 0.008 0.15847"/>
+      <origin rpy="${pi} -${pi/2} 0" xyz="-0.015639 0.008 0.15847"/>
       <parent link="${prefix}_tweezer_base_link"/>
       <child link="${prefix}_tweezer_prong_link"/>
@@ -40,5 +40,5 @@
       </visual>
       <collision>
-        <origin rpy="0 0 -${pi/2}" xyz="-0.133 0.01 0.0"/>
+        <origin rpy="${pi} 0 ${pi/2}" xyz="-0.133 0.048 0.0"/>
         <geometry>
           <mesh filename="package://micro_resector_description/meshes/tools/tweezer_right.stl" scale="0.001 0.001 0.001"/>
@@ -52,5 +52,5 @@
     <link name="${prefix}_tweezer_prong_link"/>
     <joint name="${prefix}_tweezer_joint" type="fixed">
-      <origin rpy="-${pi/2} 0 0" xyz="-0.015639 0.008 -0.15847"/>
+      <origin rpy="0 ${pi/2} 0" xyz="-0.015639 0.008 -0.15847"/>
       <parent link="${prefix}_tweezer_base_link"/>
       <child link="${prefix}_tweezer_prong_link"/>
