Commit message: removed collision from brain slice

File: urdf/samples/brain_slice.urdf.xacro (robot description, xacro)
@@ -15,10 +15,10 @@
         <material name="white"/>
         </visual>
-        <collision>
-        <origin rpy="0 0 0" xyz="0 0 0"/>
-        <geometry>
-            <mesh filename="package://micro_resector_description/meshes/samples/brain_slice.stl" scale="0.002 0.002 0.002"/>
-        </geometry>
-        </collision>
+<!--        <collision>-->
+<!--        <origin rpy="0 0 0" xyz="0 0 0"/>-->
+<!--        <geometry>-->
+<!--            <mesh filename="package://micro_resector_description/meshes/samples/brain_slice.stl" scale="0.002 0.002 0.002"/>-->
+<!--        </geometry>-->
+<!--        </collision>-->
     </link>
     <gazebo reference="brain_slice_base_link">
