Commit message: remade urdfs with reinforced tweezer and updated tool holder

File: urdf/tools/tool_holder.xacro (robot description, xacro)
@@ -25,5 +25,5 @@
             <parent link="${name}_tool_holder_link"/>
             <child link="${name}_tool_attachment_link"/>
-            <origin xyz="-0.067062 -0.006575 0.003" rpy="${pi} 0 ${-159.0 * pi/180}"/>
+            <origin xyz="-0.065195 -0.005859 0.003" rpy="${pi} 0 ${-159.0 * pi/180}"/>
         </joint>
         <link name="${name}_tool_attachment_link"/>

File: urdf/tweezer_system.xacro (robot description, xacro)
@@ -3,5 +3,5 @@
     <xacro:include filename="$(find micro_resector_description)/urdf/stage/linear_stage.xacro"/>
     <xacro:include filename="$(find micro_resector_description)/urdf/link/l_bracket.xacro"/>
-    <xacro:include filename="$(find micro_resector_description)/urdf/tools/tweezer.xacro"/>
+    <xacro:include filename="$(find micro_resector_description)/urdf/tools/tweezer_reinforced.xacro"/>
     <xacro:include filename="$(find micro_resector_description)/urdf/tools/tool_holder.xacro"/>
     <xacro:macro name="tweezer_system" params="hardware_interface name">
