Commit message: Modified starting zero position for rotation stage according to the homing procedure

File: urdf/stage/rotation_stage.xacro (robot description, xacro)
@@ -45,5 +45,5 @@
   </link>
   <joint name="${prefix}_rot_joint" type="continuous">
-    <origin rpy="0 0 0" xyz="0.0 0.015 0.0"/>
+    <origin rpy="0 ${pi/4} 0" xyz="0.0 0.015 0.0"/>
     <parent link="${prefix}_rot_base_link"/>
     <child link="${prefix}_rot_stage_link"/>
